File: KiCAD/Nodes/NodesBoosterPack.kicad_pcb (KiCad board)
At the start: 2 copper layers, 50 x 45 mm, 19 parts

Commit message: Preliminary commit - Nodes PCB
Parts:
- removed BH1750: BH1750, Pin_Headers:Pin_Header_Straight_1x05
- removed BMP180: BMP180, Pin_Headers:Pin_Header_Straight_1x04
- added LUX: BH1750, Pin_Headers:Pin_Header_Straight_1x05, F.Cu at (135.1, 77.8)
- added PRES+TEMP: BMP180, Pin_Headers:Pin_Header_Straight_1x04, F.Cu at (138.9, 85.4)
- moved G*** 15.3 mm to (145.3, 90.3)
- moved G*** 12.2 mm to (108.5, 89.5)
- moved 2xAA BAT 0.18 mm to (144.0, 93.7)
- moved ? 0.18 mm to (109.0, 80.4)
- moved ICSP 0.18 mm to (119.9, 69.3)
- moved XTAL 0.18 mm to (121.4, 65.1)
- moved C1 0.18 mm to (129.0, 63.4)
- moved C2 0.18 mm to (129.0, 56.7)
- moved D1 0.18 mm to (141.4, 58.2)
- moved G*** 0.18 mm to (145.3, 55.7)
- moved R1 0.18 mm to (122.3, 59.0)
- moved RADIO 0.18 mm to (105.0, 53.6)
- moved ? 0.18 mm to (141.4, 69.0)
- moved C3 0.18 mm to (129.0, 78.3)
- moved DHT22 0.18 mm to (114.9, 70.5)
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Routing:
- net /MISO: track 49.9 -> 59.9 mm, vias 0 -> 1
- net GND: track 144.0 -> 136.8 mm, vias 0 -> 1
- net /MOSI: track 47.0 -> 53.1 mm
- net /CE: track 90.4 -> 95.2 mm
- net /SCLK: track 72.8 -> 70.6 mm
- net /CS: track 52.4 -> 53.3 mm
- net VCC: track 103.1 -> 103.7 mm
Other:
- board text added: "FARUSAC"
- board text added: "NODO WSN"
- board text removed: "Arquitectura"
- board text removed: "Nodo WSN"
- board text removed: "USAC"
